Commit message: fix:fix ik

File: demo/kuavo-ros-controldev/src/kuavo_assets/models/biped_s45/urdf/drake/biped_v3_arm.urdf (robot description, URDF)
Before this commit: robot biped_v3_arm, 15 links, 14 joints
Links:
- added link base_link
Joints:
- added joint base_link_to_torso: type fixed, parent base_link, child torso, origin xyz=0 0 0 rpy=0 0 0
